Commit message: V1 Finish

File: usd/bottle0/urdf/bottle.urdf (robot description, URDF)
Before this commit: robot box, 1 links, 0 joints
Links:
- link base_link: mass 0.142440868845747 -> 0.0137729793309302; geometry collision mesh filename=package://bottle/meshes/base_link.STL; visual mesh filename=package://bottle/meshes/base_link.STL

File: usd/box0/urdf/box.urdf (robot description, URDF)
Before this commit: robot box, 1 links, 0 joints
Links:
- link base_link: mass 0.142440868845747 -> 0
